Commit message: 夹爪正确运动到物体上方,姿态正确

File: src/ts_robot_description/urdf/gripper.xacro (robot description, xacro)
@@ -51,5 +51,6 @@
     <parent link="ag95_base_link"/>
     <child link="grasp_link"/>
-    <origin rpy="1.5707963267948966 -1.5707963267948966 0" xyz="0.0 0.0 0.21"/>
+    <!-- <origin rpy="1.5707963267948966 -1.5707963267948966 0" xyz="0.0 0.0 0.21"/> -->
+    <origin rpy="0.0 0.0 0.0" xyz="0.0 0.0 0.21"/>
   </joint>
   <link name="left_outer_knuckle">
